File: PCB/FilaBoss_control_PCB/FilaBoss_control_PCB.kicad_sch (KiCad schematic)
At the start: 46 parts, among them J1 Encoder, J10 Power 3.3v, J11 SCL/SDA, J12 power 12v, J13 power 5v, J14 Fan connector, J15 power 12v, J16 Screen, J2 SPOOL, J3 PULLER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

Commit message: pcb v2
Parts:
- removed J16: Screen, Connector_JST:JST_PH_B4B-PH-K_1x04_P2.00mm_Vertical, symbol PCM_SparkFun-Connector:Conn_01x04_JST_P2.0mm_Vertical_PTH
- removed J9: Conn_01x04_Pot, Connector_JST:JST_PH_B4B-PH-K_1x04_P2.00mm_Vertical, symbol PCM_SparkFun-Connector:Conn_01x04_JST_P2.0mm_Vertical_PTH
- removed R14: 4.7k, Resistor_THT:R_Axial_DIN0207_L6.3mm_D2.5mm_P10.16mm_Horizontal, symbol Device:R
- removed SW1: RotaryEncoder_Switch, symbol Device:RotaryEncoder_Switch
- added D4, D5, D6: LED, symbol Device:LED
- added J16: Load, Connector_JST:JST_XA_B02B-XASK-1_1x02_P2.50mm_Vertical, symbol PCM_SparkFun-Connector:Conn_01x02_JST_P2.0mm_Horizontal_SMD
- added J17: manual, Connector_JST:JST_XA_B02B-XASK-1_1x02_P2.50mm_Vertical, symbol PCM_SparkFun-Connector:Conn_01x02_JST_P2.0mm_Horizontal_SMD
- added J18: Control leds, Connector_JST:JST_XA_B04B-XASK-1_1x04_P2.50mm_Vertical, symbol PCM_SparkFun-Connector:Conn_01x04_JST_P2.0mm_Vertical_PTH
- added J9: Extruder, Connector_JST:JST_XA_B02B-XASK-1_1x02_P2.50mm_Vertical, symbol PCM_SparkFun-Connector:Conn_01x02_JST_P2.0mm_Horizontal_SMD
- added OC1: H11A1, PCM_Package_DIP_AKL:DIP-6_W7.62mm_LongPads, symbol PCM_Optocoupler_AKL:H11A1
- added R10: 4.7k, Resistor_THT:R_Axial_DIN0207_L6.3mm_D2.5mm_P10.16mm_Horizontal, symbol Device:R
- added R11: 330R, Resistor_THT:R_Axial_DIN0207_L6.3mm_D2.5mm_P10.16mm_Horizontal, symbol Device:R
- added R12, R13: 220R, Resistor_THT:R_Axial_DIN0207_L6.3mm_D2.5mm_P10.16mm_Horizontal, symbol Device:R
- added SW1, SW2: SW_SPDT, symbol Switch:SW_SPDT
- J1: footprint Connector_JST:JST_PH_B4B-PH-K_1x04_P2.00mm_Vertical -> Connector_JST:JST_XA_B04B-XASK-1_1x04_P2.50mm_Vertical
- J11: value SCL/SDA -> SDA/SCL; footprint Connector_JST:JST_PH_B2B-PH-K_1x02_P2.00mm_Vertical -> Connector_JST:JST_XA_B02B-XASK-1_1x02_P2.50mm_Vertical
- J15: value power 12v -> power 24v
- J4: value RX/TX -> Conn_01x02_Pin; footprint Connector_JST:JST_PH_B2B-PH-K_1x02_P2.00mm_Vertical -> Connector_JST:JST_XA_B02B-XASK-1_1x02_P2.50mm_Vertical; symbol PCM_SparkFun-Connector:Conn_01x02_JST_P2.0mm_Horizontal_SMD -> Connector:Conn_01x02_Pin
- J5: value Barrel_Jack_SMD -> Screw_Terminal_01x02_P5mm; footprint PCM_SparkFun-Connector:Barrel_Jack_SMD -> TerminalBlock:TerminalBlock_MaiXu_MX126-5.0-02P_1x02_P5.00mm; symbol PCM_SparkFun-Connector:Barrel_Jack_SMD -> PCM_fab:Screw_Terminal_01x02_P5mm
- J8: footprint Connector_JST:JST_PH_B3B-PH-K_1x03_P2.00mm_Vertical -> Connector_JST:JST_XA_B03B-XASK-1_1x03_P2.50mm_Vertical
- R5: value 100R -> 220R
- R6, R7, R8, R9: value 100R -> 330R
Connections:
- net +3.3V: now also J10.1 (Pin_1), OC1.6, R10.1; no longer J10.2 (Pin_2)
- net GND: now also J10.2 (Pin_2), J5.2 (Pin_2), D4.1 (K), D5.1 (K), D6.1 (K), J16.2 (+), J17.2 (+), J18.4 (Pin_4), OC1.5, SW1.2 (B), SW2.2 (B); no longer J10.1 (Pin_1), J5.GND
- net LINE: now also J5.1 (Pin_1); no longer J5.PWR
- net at R7.1: now also U1.16 (GPIO39); no longer U1.30 (GPIO18)
- net at R15.1, R7.2: now also J16.1 (-), SW2.1 (A)
- net at R18.1, R9.1: now also J8.2; no longer J8.1
- net at R17.1, R8.1: now also J8.1; no longer J8.2
- net at R5.2: now also D4.2 (A), J18.3 (Pin_3)
- net at R16.1, R6.2: now also J17.1 (-), SW1.1 (A)
- net at U1.17 (GPIO36): now also R6.1
- net at U1.23 (GPIO15): now also A1.16 (DIR); no longer A1.15 (STEP)
- net at U1.24 (GPIO2): now also A1.15 (STEP); no longer A1.16 (DIR)
- net at U1.26 (GPIO4): now also R13.1
- net at U1.29 (GPIO5): no longer R5.1
- net at U1.31 (GPIO19): now also R5.1; no longer R6.1
- net at U1.37 (GPIO23): now also R11.2
- new net: J9.1 (-), OC1.1
- new net: J9.2 (+), OC1.2
- new net: OC1.4, R10.2, R11.1
- new net: R12.1, U1.30 (GPIO18)
- new net: D6.2 (A), J18.1 (Pin_1), R13.2
- new net: D5.2 (A), J18.2 (Pin_2), R12.2
Other:
- moved on the sheet: C3, D1, D2, J1, J14, J2, J3, J8, M1, M2, Q1, Q2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

Commit message: pcb documentation
Parts:
- added SW3: Limit_SW, symbol Switch:SW_SPDT
- J11, J16, J17, J2, J3, J9: symbol PCM_SparkFun-Connector:Conn_01x02_JST_P2.0mm_Horizontal_SMD -> Connector:Conn_01x02_Pin
- J5: value Screw_Terminal_01x02_P5mm -> Power
- J8: symbol PCM_SparkFun-Connector:Conn_01x03_JST_P2.0mm_Vertical_PTH -> Connector:Conn_01x03_Pin
Connections:
- net +3.3V: now also J10.2 (Pin_2); no longer J10.1 (Pin_1)
- net GND: now also J10.1 (Pin_1), SW3.2 (B); no longer J10.2 (Pin_2)
- net at J8.2 (Pin_2), R18.1, R9.1: now also SW3.1 (A)
- net at J8.1 (Pin_1), R17.1, R8.1: now also SW3.3 (C)

Commit message: tmc2209v2 pcb updates
Parts:
- removed D6: LED, symbol Device:LED
- added DZ1: 1N4728A, PCM_Diode_THT_AKL:D_DO-41_SOD81_P10.16mm_Horizontal_Zener, symbol PCM_Diode_Zener_AKL:1N4728A
- added R14: 1K, Resistor_THT:R_Axial_DIN0207_L6.3mm_D2.5mm_P10.16mm_Horizontal, symbol Device:R
- added R19: 330R, Resistor_THT:R_Axial_DIN0207_L6.3mm_D2.5mm_P10.16mm_Horizontal, symbol Device:R
- A1: symbol Driver_Motor:Pololu_Breakout_A4988 -> custom:tmc2209v2
- J10, J12, J13, J15: footprint TerminalBlock:TerminalBlock_Xinya_XY308-2.54-2P_1x02_P2.54mm_Horizontal -> TerminalBlock:TerminalBlock_MaiXu_MX126-5.0-02P_1x02_P5.00mm
- J18: footprint Connector_JST:JST_XA_B04B-XASK-1_1x04_P2.50mm_Vertical -> Connector_JST:JST_XA_B04B-XASK-1_1x03_P2.50mm_Vertical; symbol PCM_SparkFun-Connector:Conn_01x04_JST_P2.0mm_Vertical_PTH -> PCM_SparkFun-Connector:Conn_01x03_P2.54mm_Locking
- R13: value 220R -> 4.7k
Connections:
- net +3.3V: now also R13.1, DZ1.1 (K); no longer A1.10 (MS1), A1.11 (MS2), A1.12 (MS3), A1.13 (~{RESET}), A1.14 (~{SLEEP})
- net GND: now also A1.10 (MS1), A1.11 (MS2), J18.3 (Pin_3), DZ1.2 (A); no longer J18.4 (Pin_4)
- net at J14.2 (Pin_2): now also R13.2, R19.1; no longer U1.13 (GPIO32)
- net at U1.23 (GPIO15): now also A1.15 (STEP); no longer A1.16 (DIR)
- net at U1.24 (GPIO2): no longer A1.15 (STEP)
- net at U1.26 (GPIO4): now also R14.1; no longer R13.1
- net at U1.5 (GPIO13): now also A1.14 (UART), R14.2
- net at U1.7 (GPIO12): now also A1.16 (DIR)
- net at J18.1 (Pin_1): now also D5.2 (A), R12.2; no longer R13.2
- net at D4.2 (A), R5.2: now also J18.2 (Pin_2); no longer J18.3 (Pin_3)
- new net: R19.2, U1.13 (GPIO32)
Other:
- moved on the sheet: A1, J1, J14, J7

Commit message: pcb WIP
Parts:
- added R20: 2k, Resistor_THT:R_Axial_DIN0207_L6.3mm_D2.5mm_P10.16mm_Horizontal, symbol Device:R
- R19: value 330R -> 1k
Connections:
- net +3.3V: no longer R13.1
- net +5V: now also R13.1
- net GND: now also R20.2
- net at R19.2, U1.13 (GPIO32): now also R20.1
Other:
- moved on the sheet: R19
Changed lines of the file:
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@@
 	)
 	(junction
+		(at 119.38 125.73)
+		(diameter 0)
+		(color 0 0 0 0)
+	)
+	(junction
 		(at 68.58 149.86)
 		(diameter 0)
@@
 	(wire
 		(pts
+			(xy 119.38 127) (xy 119.38 125.73)
+		)
+		(stroke
+			(width 0)
+			(type default)
+		)
+	)
+	(wire
+		(pts
 			(xy 101.6 67.31) (xy 101.6 71.12)
 		)
@@
 	(wire
 		(pts
+			(xy 119.38 125.73) (xy 142.24 125.73)
+		)
+		(stroke
+			(width 0)
+			(type default)
+		)
+	)
+	(wire
+		(pts
 			(xy 69.85 129.54) (xy 69.85 137.16)
 		)
@@
 	(wire
 		(pts
-			(xy 111.76 125.73) (xy 115.57 125.73)
-		)
-		(stroke
-			(width 0)
-			(type default)
-		)
-	)
-	(wire
-		(pts
 			(xy 232.41 109.22) (xy 194.31 109.22)
 		)
@@
 		)
 	)
-	(wire
-		(pts
-			(xy 123.19 125.73) (xy 142.24 125.73)
-		)
-		(stroke
-			(width 0)
-			(type default)
-		)
-	)
 	(symbol
 		(lib_id "power:+12V")
@@
 		)
 		(property "Value" "GND"
-			(at 97.79 133.35 90)
+			(at 102.87 130.81 90)
 			(effects
 				(font
@@
 	)
 	(symbol
-		(lib_id "power:+3.3V")
-		(at 111.76 134.62 0)
-		(mirror x)
-		(unit 1)
-		(exclude_from_sim no)
-		(in_bom yes)
-		(on_board yes)
-		(dnp no)
-		(property "Reference" "#PWR054"
-			(at 111.76 130.81 0)
-			(effects
-				(font
-					(size 1.27 1.27)
-				)
-				(hide yes)
-			)
-		)
-		(property "Value" "+3.3V"
-			(at 111.76 138.43 0)
-			(effects
-				(font
-					(size 1.27 1.27)
-				)
-			)
-		)
-		(property "Footprint" ""
-			(at 111.76 134.62 0)
-			(effects
-				(font
-					(size 1.27 1.27)
-				)
-				(hide yes)
-			)
-		)
-		(property "Datasheet" ""
-			(at 111.76 134.62 0)
-			(effects
-				(font
-					(size 1.27 1.27)
-				)
-				(hide yes)
-			)
-		)
-		(property "Description" "Power symbol creates a global label with name \"+3.3V\""
-			(at 111.76 134.62 0)
-			(effects
-				(font
-					(size 1.27 1.27)
-				)
-				(hide yes)
-			)
-		)
-		(pin "1"
-		)
-		(instances
-			(project "FilaBoss_control_PCB"
-				(path "/2f49582a-29fd-468d-b48c-a2b14259075d"
-					(reference "#PWR054")
-					(unit 1)
-				)
-			)
-		)
-	)
-	(symbol
 		(lib_id "Connector:Conn_01x03_Pin")
 		(at 107.95 99.06 0)
@@
 	)
 	(symbol
+		(lib_id "power:+5V")
+		(at 111.76 134.62 180)
+		(unit 1)
+		(exclude_from_sim no)
+		(in_bom yes)
+		(on_board yes)
+		(dnp no)
+		(property "Reference" "#PWR054"
+			(at 111.76 130.81 0)
+			(effects
+				(font
+					(size 1.27 1.27)
+				)
+				(hide yes)
+			)
+		)
+		(property "Value" "+5V"
+			(at 111.76 138.43 0)
+			(effects
+				(font
+					(size 1.27 1.27)
+				)
+			)
+		)
+		(property "Footprint" ""
+			(at 111.76 134.62 0)
+			(effects
+				(font
+					(size 1.27 1.27)
+				)
+				(hide yes)
+			)
+		)
+		(property "Datasheet" ""
+			(at 111.76 134.62 0)
+			(effects
+				(font
+					(size 1.27 1.27)
+				)
+				(hide yes)
+			)
+		)
+		(property "Description" "Power symbol creates a global label with name \"+5V\""
+			(at 111.76 134.62 0)
+			(effects
+				(font
+					(size 1.27 1.27)
+				)
+				(hide yes)
+			)
+		)
+		(pin "1"
+		)
+		(instances
+			(project "FilaBoss_control_PCB"
+				(path "/2f49582a-29fd-468d-b48c-a2b14259075d"
+					(reference "#PWR054")
+					(unit 1)
+				)
+			)
+		)
+	)
+	(symbol
 		(lib_id "power:+12V")
 		(at 77.47 35.56 270)
@@
 	(symbol
 		(lib_id "Device:R")
-		(at 119.38 125.73 90)
+		(at 115.57 125.73 90)
 		(unit 1)
 		(exclude_from_sim no)
@@
 		(dnp no)
 		(property "Reference" "R19"
-			(at 121.92 124.46 90)
+			(at 118.11 124.46 90)
 			(effects
 				(font
@@
 			)
 		)
-		(property "Value" "330R"
-			(at 116.84 125.73 90)
+		(property "Value" "1k"
+			(at 114.3 125.73 90)
 			(effects
 				(font
@@
 		)
 		(property "Footprint" "Resistor_THT:R_Axial_DIN0207_L6.3mm_D2.5mm_P10.16mm_Horizontal"
-			(at 119.38 127.508 90)
+			(at 115.57 127.508 90)
 			(effects
 				(font
@@
 		)
 		(property "Datasheet" "~"
-			(at 119.38 125.73 0)
+			(at 115.57 125.73 0)
 			(effects
 				(font
@@
 		)
 		(property "Description" "Resistor"
-			(at 119.38 125.73 0)
+			(at 115.57 125.73 0)
 			(effects
 				(font
@@
 	)
 	(symbol
+		(lib_id "Device:R")
+		(at 119.38 130.81 0)
+		(unit 1)
+		(exclude_from_sim no)
+		(in_bom yes)
+		(on_board yes)
+		(dnp no)
+		(property "Reference" "R20"
+			(at 121.92 129.54 90)
+			(effects
+				(font
+					(size 1.27 1.27)
+				)
+				(justify right)
+			)
+		)
+		(property "Value" "2k"
+			(at 119.38 129.54 90)
+			(effects
+				(font
+					(size 1.27 1.27)
+				)
+				(justify right)
+			)
+		)
+		(property "Footprint" "Resistor_THT:R_Axial_DIN0207_L6.3mm_D2.5mm_P10.16mm_Horizontal"
+			(at 117.602 130.81 90)
+			(effects
+				(font
+					(size 1.27 1.27)
+				)
+				(hide yes)
+			)
+		)
+		(property "Datasheet" "~"
+			(at 119.38 130.81 0)
+			(effects
+				(font
+					(size 1.27 1.27)
+				)
+				(hide yes)
+			)
+		)
+		(property "Description" "Resistor"
+			(at 119.38 130.81 0)
+			(effects
+				(font
+					(size 1.27 1.27)
+				)
+				(hide yes)
+			)
+		)
+		(pin "2"
+		)
+		(pin "1"
+		)
+		(instances
+			(project "FilaBoss_control_PCB"
+				(path "/2f49582a-29fd-468d-b48c-a2b14259075d"
+					(reference "R20")
+					(unit 1)
+				)
+			)
+		)
+	)
+	(symbol
 		(lib_id "power:+3.3V")
 		(at 160.02 88.9 90)
@@
 					(unit 1)
 				)
+			)
+		)
+	)
+	(symbol
+		(lib_id "power:GND")
+		(at 119.38 134.62 0)
+		(unit 1)
+		(exclude_from_sim no)
+		(in_bom yes)
+		(on_board yes)
+		(dnp no)
+		(property "Reference" "#PWR055"
+			(at 119.38 140.97 0)
+			(effects
+				(font
+					(size 1.27 1.27)
+				)
+				(hide yes)
+			)
+		)
+		(property "Value" "GND"
+			(at 119.38 138.43 0)
+			(effects
+				(font
+					(size 1.27 1.27)
+				)
+			)
+		)
+		(property "Footprint" ""
+			(at 119.38 134.62 0)
+			(effects
+				(font
+					(size 1.27 1.27)
+				)
+				(hide yes)
+			)
+		)
+		(property "Datasheet" ""
+			(at 119.38 134.62 0)
+			(effects
+				(font
+					(size 1.27 1.27)
+				)
+				(hide yes)
+			)
+		)
+		(property "Description" "Power symbol creates a global label with name \"GND\" , ground"
+			(at 119.38 134.62 0)
+			(effects
+				(font
+					(size 1.27 1.27)
+				)
+				(hide yes)
+			)
+		)
+		(pin "1"
+		)
+		(instances
+			(project "FilaBoss_control_PCB"
+				(path "/2f49582a-29fd-468d-b48c-a2b14259075d"
+					(reference "#PWR055")
+					(unit 1)
+				)

Commit message: pcb v3
Parts:
- removed C3: C, Capacitor_THT:C_Axial_L5.1mm_D3.1mm_P10.00mm_Horizontal, symbol Device:C
- removed DZ1: 1N4728A, PCM_Diode_THT_AKL:D_DO-41_SOD81_P10.16mm_Horizontal_Zener, symbol PCM_Diode_Zener_AKL:1N4728A
- added C1: C, Capacitor_THT:C_Axial_L5.1mm_D3.1mm_P7.50mm_Horizontal, symbol Device:C
- added D6: 1.5KE36CA, PCM_Diode_THT_AKL:D_DO-201_P12.70mm_Horizontal_TVS, symbol PCM_Diode_TVS_AKL:1.5KE36CA
- added DZ1: 1EZ15, PCM_Diode_THT_AKL:D_DO-41_SOD81_P10.16mm_Horizontal_Zener, symbol PCM_Diode_Zener_AKL:1EZ15
- added Q3: IRF9540N, PCM_Package_TO_SOT_THT_AKL:TO-220-3_Vertical_GDS, symbol PCM_Transistor_MOSFET_AKL:IRF9540N
- added R21: 4.7k, Resistor_THT:R_Axial_DIN0207_L6.3mm_D2.5mm_P10.16mm_Horizontal, symbol Device:R
- added R22: 2k, Resistor_THT:R_Axial_DIN0207_L6.3mm_D2.5mm_P10.16mm_Horizontal, symbol Device:R
- J18: footprint Connector_JST:JST_XA_B04B-XASK-1_1x03_P2.50mm_Vertical -> Connector_JST:JST_XA_B03B-XASK-1_1x03_P2.50mm_Vertical
- J4: value Conn_01x02_Pin -> RX/TX
- R12, R5: value 220R -> 330R
- U4: value R-78E12-2 -> R-78B12-2.0; footprint Converter_DCDC:Converter_DCDC_RECOM_R-78E-0.5_THT -> Converter_DCDC:Converter_DCDC_RECOM_R-78B-2.0_THT; symbol Converter_DCDC:R-78E5.0-0.5 -> Converter_DCDC:R-78B12-2.0
Connections:
- net +24V: now also D6.2 (A)
- net +3.3V: now also C1.1
- net GND: now also J5.1 (Pin_1), C1.2, D6.1 (K), R22.1; no longer J5.2 (Pin_2)
- net LINE: now also J5.2 (Pin_2); no longer J5.1 (Pin_1)
- net VDC: now also Q3.2 (D); no longer L1.1
- net at OC1.1: now also R21.1; no longer J9.1 (Pin_1)
- net at J8.2 (Pin_2), R18.1, R9.1: now also SW3.3 (C); no longer SW3.1 (A)
- net at J8.1 (Pin_1), R17.1, R8.1: now also SW3.1 (A); no longer SW3.3 (C)
- net at U1.10 (GPIO26): now also J4.2 (Pin_2); no longer R1.2
- net at U1.11 (GPIO25): now also J4.1 (Pin_1); no longer R4.2
- net at U1.23 (GPIO15): now also A1.16 (DIR); no longer A1.15 (STEP)
- net at U1.26 (GPIO4): now also A1.15 (STEP); no longer R14.1
- net at U1.27 (GPIO16/RX2): now also A1.14 (UART), R14.2; no longer J4.1 (Pin_1)
- net at U1.28 (GPIO17/TX2): now also R14.1; no longer J4.2 (Pin_2)
- net at U1.7 (GPIO12): now also R4.2; no longer A1.16 (DIR)
- new net: R1.2, U1.5 (GPIO13)
- new net: J9.1 (Pin_1), R21.2
- new net: DZ1.2 (A), Q3.1 (G), R22.2
- new net VCC: DZ1.1 (K), L1.1, Q3.3 (S)
Other:
- moved on the sheet: C2, D1, D2, D3, D4, D5, F1, J1, J14, J16, J17, J18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

Commit message: pcb v4
Parts:
- added R23: 4.7k, Resistor_THT:R_Axial_DIN0207_L6.3mm_D2.5mm_P10.16mm_Horizontal, symbol Device:R
- added R24, R25: 330R, Resistor_THT:R_Axial_DIN0207_L6.3mm_D2.5mm_P10.16mm_Horizontal, symbol Device:R
- D6: value 1.5KE36CA -> TVS
- F1: footprint Fuse:Fuseholder_Clip-5x20mm_Littelfuse_521_Lateral_P17.00x5.00mm_D1.30mm_Horizontal -> fuse:fuse
- Q3: value IRF9540N -> Power Pmos
- R19: value 1k -> 330R
- R20: value 2k -> 4.7k
Connections:
- net +3.3V: now also J10.1 (Pin_1), R13.1, R20.2, R23.2; no longer J10.2 (Pin_2)
- net +5V: now also J1.3 (Pin_3); no longer J1.2 (Pin_2), R13.1
- net GND: now also J1.4 (Pin_4), J10.2 (Pin_2), J5.2 (Pin_2); no longer J1.1 (Pin_1), J10.1 (Pin_1), J5.1 (Pin_1), R20.2
- net LINE: now also J5.1 (Pin_1); no longer J5.2 (Pin_2)
- net at U1.10 (GPIO26): now also J4.1 (Pin_1); no longer J4.2 (Pin_2)
- net at U1.11 (GPIO25): now also J4.2 (Pin_2); no longer J4.1 (Pin_1)
- net at R19.2, U1.13 (GPIO32): no longer R20.1
- net at U1.8 (GPIO14): now also R25.2; no longer J1.3 (Pin_3)
- net at U1.9 (GPIO27): now also R24.2; no longer J1.4 (Pin_4)
- new net: J1.2 (Pin_2), R23.1, R25.1
- new net: J1.1 (Pin_1), R20.1, R24.1
Other:
- moved on the sheet: A1, D1, D2, J1, J14, J2, J3, J5, J7, M1, M2, Q1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

Commit message: -
Parts:
- Q3: value Power Pmos -> IRF9540N
- R22: value 2k -> 1k
Changed lines of the file:
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@@
 		(dnp no)
 		(property "Reference" "Q3"
-			(at 48.26 17.78 90)
+			(at 50.8 19.05 0)
 			(effects
 				(font
@@
 			)
 		)
-		(property "Value" "Power Pmos"
-			(at 43.18 15.24 90)
+		(property "Value" "IRF9540N"
+			(at 48.26 19.05 0)
 			(effects
 				(font
@@
 			)
 		)
-		(property "Value" "2k"
+		(property "Value" "1k"
 			(at 50.8 34.29 90)
 			(effects
