File: PCB/FilaBoss_control_PCB/FilaBoss_control_PCB.kicad_pcb (KiCad board)
At the start: 2 copper layers, 101.6 x 80 mm, 43 parts, among them J1 Encoder, J10 Power 3.3v, J11 SCL/SDA, J12 power 12v, J13 power 5v, J14 Fan connector, J15 power 12v, J16 Screen, J2 SPOOL, J3 PULLER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

Commit message: pcb v2
Parts:
- removed R14: 4.7k, Resistor_THT:R_Axial_DIN0207_L6.3mm_D2.5mm_P10.16mm_Horizontal
- added J17: manual, Connector_JST:JST_XA_B02B-XASK-1_1x02_P2.50mm_Vertical, F.Cu at (102.2, 166.4)
- added J18: Control leds, Connector_JST:JST_XA_B04B-XASK-1_1x04_P2.50mm_Vertical, F.Cu at (95.8, 91.4)
- added OC1: H11A1, PCM_Package_DIP_AKL:DIP-6_W7.62mm_LongPads, F.Cu at (86.4, 109.9)
- added R10: 4.7k, Resistor_THT:R_Axial_DIN0207_L6.3mm_D2.5mm_P10.16mm_Horizontal, F.Cu at (91.4, 127.0)
- added R11: 330R, Resistor_THT:R_Axial_DIN0207_L6.3mm_D2.5mm_P10.16mm_Horizontal, F.Cu at (81.3, 121.9)
- added R12: 220R, Resistor_THT:R_Axial_DIN0207_L6.3mm_D2.5mm_P10.16mm_Horizontal, F.Cu at (106.7, 114.3)
- added R13: 220R, Resistor_THT:R_Axial_DIN0207_L6.3mm_D2.5mm_P10.16mm_Horizontal, F.Cu at (109.2, 106.7)
- J1: footprint Connector_JST:JST_PH_B4B-PH-K_1x04_P2.00mm_Vertical -> Connector_JST:JST_XA_B04B-XASK-1_1x04_P2.50mm_Vertical
- J11: value SCL/SDA -> SDA/SCL; footprint Connector_JST:JST_PH_B2B-PH-K_1x02_P2.00mm_Vertical -> Connector_JST:JST_XA_B02B-XASK-1_1x02_P2.50mm_Vertical
- J15: value power 12v -> power 24v
- J16: value Screen -> Load; footprint Connector_JST:JST_PH_B4B-PH-K_1x04_P2.00mm_Vertical -> Connector_JST:JST_XA_B02B-XASK-1_1x02_P2.50mm_Vertical
- J4: value RX/TX -> Conn_01x02_Pin; footprint Connector_JST:JST_PH_B2B-PH-K_1x02_P2.00mm_Vertical -> Connector_JST:JST_XA_B02B-XASK-1_1x02_P2.50mm_Vertical
- J5: value Barrel_Jack_SMD -> Screw_Terminal_01x02_P5mm; footprint PCM_SparkFun-Connector:Barrel_Jack_SMD -> TerminalBlock:TerminalBlock_MaiXu_MX126-5.0-02P_1x02_P5.00mm
- J8: footprint Connector_JST:JST_PH_B3B-PH-K_1x03_P2.00mm_Vertical -> Connector_JST:JST_XA_B03B-XASK-1_1x03_P2.50mm_Vertical
- J9: value Conn_01x04_Pot -> Extruder; footprint Connector_JST:JST_PH_B4B-PH-K_1x04_P2.00mm_Vertical -> Connector_JST:JST_XA_B02B-XASK-1_1x02_P2.50mm_Vertical
- R5: value 100R -> 220R
- R6, R7, R8, R9: value 100R -> 330R
- moved J11 84.9 mm to (72.4, 91.4), turned to 180 degrees
- moved J8 66.1 mm to (122.1, 166.4)
- moved R16 50.9 mm to (101.5, 158.5), turned to 180 degrees
- moved R18 50.7 mm to (101.5, 150.9), turned to 180 degrees
- moved R15 48.2 mm to (101.5, 154.7), turned to 180 degrees
- moved R9 48.0 mm to (115.6, 153.0), turned to 180 degrees
- moved R17 46.0 mm to (101.5, 147.1), turned to 180 degrees
- moved J4 45.7 mm to (108.0, 91.4), turned to 180 degrees
- moved J14 39.7 mm to (134.7, 158.1)
- moved R8 38.6 mm to (115.6, 149.2), turned to 180 degrees
- moved R6 37.7 mm to (105.4, 160.7), turned to 0 degrees
- moved R7 35.3 mm to (105.4, 156.8), turned to 0 degrees
- moved A1 33.7 mm to (134.6, 99.1)
- moved J9 33.7 mm to (81.6, 91.4)
- moved J13 30.4 mm to (85.4, 168.9)
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Connections:
- J10 pad 1: GND -> +3.3V
- J10 pad 2: +3.3V -> GND
- J16 pad 1: GND -> Net-(J16--)
- J16 pad 2: +3.3V -> GND
- J9 pad 1: GND -> Net-(J9--)
- J9 pad 2: Net-(J9-Pin_2) -> Net-(J9-+)
- R15 pad 1: Net-(J9-Pin_3) -> Net-(J16--)
- R16 pad 1: Net-(J9-Pin_4) -> Net-(J17--)
- R17 pad 1: Net-(J8-Pad2) -> Net-(J8-Pad1)
- R18 pad 1: Net-(J8-Pad1) -> Net-(J8-Pad2)
- R5 pad 1: Net-(U1-GPIO5) -> Net-(U1-GPIO19)
- R5 pad 2: Net-(J9-Pin_2) -> Net-(J18-Pin_3)
- R6 pad 1: Net-(U1-GPIO19) -> Net-(U1-GPIO36)
- R6 pad 2: Net-(J9-Pin_4) -> Net-(J17--)
- R7 pad 1: Net-(U1-GPIO18) -> Net-(U1-GPIO39)
- R7 pad 2: Net-(J9-Pin_3) -> Net-(J16--)
- R8 pad 1: Net-(J8-Pad2) -> Net-(J8-Pad1)
- R9 pad 1: Net-(J8-Pad1) -> Net-(J8-Pad2)
- U1 pad 16: unconnected-(U1-GPIO39-Pad16) -> Net-(U1-GPIO39)
- U1 pad 17: unconnected-(U1-GPIO36-Pad17) -> Net-(U1-GPIO36)
- U1 pad 23: Net-(A1-STEP) -> Net-(A1-DIR)
- U1 pad 24: Net-(A1-DIR) -> Net-(A1-STEP)
- U1 pad 26: unconnected-(U1-GPIO4-Pad26) -> Net-(U1-GPIO4)
- U1 pad 29: Net-(U1-GPIO5) -> unconnected-(U1-GPIO5-Pad29)
- U1 pad 37: unconnected-(U1-GPIO23-Pad37) -> Net-(U1-GPIO23)
Routing:
- net GND: track 0.00 -> 205.3 mm, vias 1 -> 8
- net +12V: track 0.00 -> 81.5 mm
- net Net-(J11--): track 83.1 -> 47.8 mm
- net Net-(A1-STEP): track 41.0 -> 8.98 mm
- net Net-(J17--): track 0.00 -> 30.6 mm
- net Net-(J16--): track 0.00 -> 28.8 mm
- net Net-(A1-DIR): track 36.4 -> 8.98 mm
- net Net-(U1-GPIO36): track 0.00 -> 26.3 mm
- net Net-(J18-Pin_2): track 0.00 -> 24.7 mm
- net Net-(U1-GPIO39): track 0.00 -> 22.5 mm
- net Net-(U1-GPIO5): track 22.3 -> 0.00 mm
- net Net-(J9-+): track 0.00 -> 20.6 mm
- net Net-(J9--): track 0.00 -> 20.4 mm
- net Net-(J18-Pin_3): track 0.00 -> 19.3 mm
- net VDC: track 0.00 -> 19.2 mm
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- removed copper zone on B.Cu, net +12V
- removed copper zone on B.Cu, net LINE
- removed copper zone on B.Cu, net VDC
Other:
- board size 101.6 x 80 mm -> 102.9 x 87.6 mm

Commit message: pcb documentation
Parts:
- J5: value Screw_Terminal_01x02_P5mm -> Power
- moved J10 2.54 mm to (130.2, 91.4), turned to 180 degrees
Connections:
- J10 pad 1: +3.3V -> GND
- J10 pad 2: GND -> +3.3V

Commit message: tmc2209v2 pcb updates
Parts:
- added DZ1: 1N4728A, PCM_Diode_THT_AKL:D_DO-41_SOD81_P10.16mm_Horizontal_Zener, F.Cu at (117.1, 70.8)
- added R14: 1K, Resistor_THT:R_Axial_DIN0207_L6.3mm_D2.5mm_P10.16mm_Horizontal, F.Cu at (109.7, 114.8)
- added R19: 330R, Resistor_THT:R_Axial_DIN0207_L6.3mm_D2.5mm_P10.16mm_Horizontal, F.Cu at (116.8, 74.9)
- J10, J12, J13, J15: footprint TerminalBlock:TerminalBlock_Xinya_XY308-2.54-2P_1x02_P2.54mm_Horizontal -> TerminalBlock:TerminalBlock_MaiXu_MX126-5.0-02P_1x02_P5.00mm
- R13: value 220R -> 4.7k
Connections:
- A1 pad 10: +3.3V -> GND
- A1 pad 11: +3.3V -> GND
- A1 pad 12: +3.3V -> unconnected-(A1-R8-Pad12)
- A1 pad 13: +3.3V -> unconnected-(A1-NC-Pad13)
- A1 pad 14: +3.3V -> Net-(A1-UART)
- J18 pad 3: Net-(J18-Pin_3) -> GND
- J18 pad 4: GND -> (no net)
- R12 pad 2: Net-(J18-Pin_2) -> Net-(J18-Pin_1)
- R13 pad 1: Net-(U1-GPIO4) -> +3.3V
- R13 pad 2: Net-(J18-Pin_1) -> Net-(J14-Pin_2)
- R5 pad 2: Net-(J18-Pin_3) -> Net-(J18-Pin_2)
- U1 pad 13: Net-(J14-Pin_2) -> Net-(U1-GPIO32)
- U1 pad 23: Net-(A1-DIR) -> Net-(A1-STEP)
- U1 pad 24: Net-(A1-STEP) -> unconnected-(U1-GPIO2-Pad24)
- U1 pad 5: unconnected-(U1-GPIO13-Pad5) -> Net-(A1-UART)
- U1 pad 7: unconnected-(U1-GPIO12-Pad7) -> Net-(A1-DIR)
Routing:
- net Net-(A1-UART): track 0.00 -> 54.9 mm
- net Net-(J18-Pin_3): track 19.3 -> 0.00 mm
- net (no net): track 0.00 -> 19.3 mm
- net Net-(U1-GPIO4): track 16.2 -> 20.8 mm

Commit message: pcb v3
Parts:
- removed C3: C, Capacitor_THT:C_Axial_L5.1mm_D3.1mm_P10.00mm_Horizontal
- added C1: C, Capacitor_THT:C_Axial_L5.1mm_D3.1mm_P7.50mm_Horizontal, F.Cu at (86.4, 121.9)
- added D6: 1.5KE36CA, PCM_Diode_THT_AKL:D_DO-201_P12.70mm_Horizontal_TVS, F.Cu at (43.2, 152.2)
- added Q3: IRF9540N, PCM_Package_TO_SOT_THT_AKL:TO-220-3_Vertical_GDS, F.Cu at (67.4, 160.9)
- added R20: 2k, Resistor_THT:R_Axial_DIN0207_L6.3mm_D2.5mm_P10.16mm_Horizontal, F.Cu at (115.1, 149.4)
- added R21: 4.7k, Resistor_THT:R_Axial_DIN0207_L6.3mm_D2.5mm_P10.16mm_Horizontal, F.Cu at (83.8, 106.7)
- added R22: 2k, Resistor_THT:R_Axial_DIN0207_L6.3mm_D2.5mm_P10.16mm_Horizontal, F.Cu at (67.4, 148.1)
- DZ1: value 1N4728A -> 1EZ15
- J18: footprint Connector_JST:JST_XA_B04B-XASK-1_1x04_P2.50mm_Vertical -> Connector_JST:JST_XA_B03B-XASK-1_1x03_P2.50mm_Vertical
- J4: value Conn_01x02_Pin -> RX/TX
- R12, R5: value 220R -> 330R
- R19: value 330R -> 1k
- U4: value R-78E12-2 -> R-78B12-2.0; footprint Converter_DCDC:Converter_DCDC_RECOM_R-78E-0.5_THT -> Converter_DCDC:Converter_DCDC_RECOM_R-78B-2.0_THT
- moved R19 85.3 mm to (122.4, 160.0), turned to 90 degrees
- moved DZ1 82.6 mm to (71.4, 139.6), turned to -90 degrees
- moved J4 61.2 mm to (84.5, 147.9), turned to 90 degrees
- moved R13 55.1 mm to (139.2, 152.9)
- moved C2 14.5 mm to (63.3, 131.1), turned to 0 degrees
- moved R10 13.2 mm to (78.2, 127.5), turned to 90 degrees
- moved D3 12.1 mm to (99.7, 162.7), turned to 180 degrees
- moved A1 11.5 mm to (123.2, 97.8)
- moved R3 10.2 mm to (63.5, 122.2)
- moved R2 8.94 mm to (63.5, 118.4)
- moved J13 8.28 mm to (93.6, 168.9)
- moved U4 8.05 mm to (77.0, 154.9)
- moved J2 6.03 mm to (43.2, 122.2)
- moved J3 6.01 mm to (43.2, 131.1)
- moved J8 5.45 mm to (127.6, 166.4)
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Connections:
- DZ1 pad 1: +3.3V -> VCC
- DZ1 pad 2: GND -> Net-(DZ1-A)
- J5 pad 1: LINE -> GND
- J5 pad 2: GND -> LINE
- L1 pad 1: VDC -> VCC
- OC1 pad 1: Net-(J9-Pin_1) -> Net-(OC1-Pad1)
- R1 pad 2: Net-(U1-GPIO26) -> Net-(U1-GPIO13)
- R13 pad 1: +3.3V -> +5V
- R14 pad 1: Net-(U1-GPIO4) -> Net-(U1-GPIO17/TX2)
- R4 pad 2: Net-(U1-GPIO25) -> Net-(U1-GPIO12)
- U1 pad 10: Net-(U1-GPIO26) -> Net-(J4-Pin_2)
- U1 pad 11: Net-(U1-GPIO25) -> Net-(J4-Pin_1)
- U1 pad 23: Net-(A1-STEP) -> Net-(A1-DIR)
- U1 pad 26: Net-(U1-GPIO4) -> Net-(A1-STEP)
- U1 pad 27: Net-(J4-Pin_1) -> Net-(A1-UART)
- U1 pad 28: Net-(J4-Pin_2) -> Net-(U1-GPIO17/TX2)
- U1 pad 5: Net-(A1-UART) -> Net-(U1-GPIO13)
- U1 pad 7: Net-(A1-DIR) -> Net-(U1-GPIO12)
Routing:
- net Net-(U1-GPIO13): track 0.00 -> 46.1 mm
- net Net-(A1-UART): track 54.9 -> 9.09 mm
- net Net-(U1-GPIO12): track 0.00 -> 39.5 mm
- net Net-(U1-GPIO26): track 31.1 -> 0.00 mm
- net Net-(U1-GPIO25): track 27.0 -> 0.00 mm
- net LINE: track 21.9 -> 0.00 mm
- net Net-(U1-GPIO32): track 0.00 -> 21.7 mm
- net Net-(U1-GPIO4): track 20.8 -> 0.00 mm
- net (no net): track 19.3 -> 0.00 mm
- net VDC: track 19.2 -> 0.00 mm
- net Net-(J14-Pin_2): track 33.9 -> 17.3 mm
- net Net-(J9-Pin_1): track 20.4 -> 5.98 mm
- net Net-(DZ1-A): track 0.00 -> 12.8 mm
- net VCC: track 0.00 -> 11.9 mm
- net +3.3V: track 16.0 -> 7.21 mm
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- added copper zone on B.Cu, net GND
- added copper zone on B.Cu, net LINE
- added copper zone on F.Cu, net LINE
- added copper zone on B.Cu, net VCC
- added copper zone on B.Cu, net VDC
- added copper zone on F.Cu, net VDC

Commit message: pcb v4
Parts:
- added R23: 4.7k, Resistor_THT:R_Axial_DIN0207_L6.3mm_D2.5mm_P10.16mm_Horizontal, F.Cu at (135.3, 133.3)
- added R24: 330R, Resistor_THT:R_Axial_DIN0207_L6.3mm_D2.5mm_P10.16mm_Horizontal, F.Cu at (125.7, 130.2)
- added R25: 330R, Resistor_THT:R_Axial_DIN0207_L6.3mm_D2.5mm_P10.16mm_Horizontal, F.Cu at (128.3, 133.3)
- D6: value 1.5KE36CA -> TVS
- F1: footprint Fuse:Fuseholder_Clip-5x20mm_Littelfuse_521_Lateral_P17.00x5.00mm_D1.30mm_Horizontal -> fuse:fuse
- Q3: value IRF9540N -> Power Pmos
- R19: value 1k -> 330R
- R20: value 2k -> 4.7k
- moved J4 50.2 mm to (134.6, 150.4), turned to 180 degrees
- moved R13 50.2 mm to (90.2, 142.2), turned to 0 degrees
- moved R20 28.8 mm to (139.1, 133.3), turned to 90 degrees
- moved Q3 28.2 mm to (49.5, 139.1), turned to 0 degrees
- moved R19 25.2 mm to (102.9, 144.1), turned to 0 degrees
- moved D6 23.6 mm to (66.7, 149.9), turned to -90 degrees
- moved C2 17.5 mm to (75.6, 143.5)
- moved J5 16.9 mm to (55.7, 168.9), turned to 0 degrees
- moved L1 15.3 mm to (48.3, 152.4), turned to 0 degrees
- moved R22 14.1 mm to (74.9, 136.1), turned to 180 degrees
- moved F1 13.1 mm to (42.3, 154.9), turned to 90 degrees
- moved DZ1 12.3 mm to (59.1, 139.4), turned to 0 degrees
- moved J11 11.4 mm to (83.8, 91.4)
- moved J9 11.1 mm to (92.7, 91.4)
- moved J18 8.38 mm to (104.1, 91.4)
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Connections:
- J1 pad 1: GND -> Net-(J1-Pin_1)
- J1 pad 2: +5V -> Net-(J1-Pin_2)
- J1 pad 3: Net-(J1-Pin_3) -> +5V
- J1 pad 4: Net-(J1-Pin_4) -> GND
- J10 pad 1: GND -> +3.3V
- J10 pad 2: +3.3V -> GND
- J5 pad 1: GND -> LINE
- J5 pad 2: LINE -> GND
- R13 pad 1: +5V -> +3.3V
- R20 pad 1: Net-(U1-GPIO32) -> Net-(J1-Pin_1)
- R20 pad 2: GND -> +3.3V
- U1 pad 10: Net-(J4-Pin_2) -> Net-(J4-Pin_1)
- U1 pad 11: Net-(J4-Pin_1) -> Net-(J4-Pin_2)
- U1 pad 8: Net-(J1-Pin_3) -> Net-(U1-GPIO14)
- U1 pad 9: Net-(J1-Pin_4) -> Net-(U1-GPIO27)
Routing:
- net GND: track 210.1 -> 137.0 mm, vias 6 -> 8
- net Net-(J1-Pin_1): track 0.00 -> 26.5 mm
- net Net-(J14-Pin_2): track 17.3 -> 40.8 mm
- net Net-(J1-Pin_2): track 0.00 -> 20.9 mm
- net Net-(J18-Pin_1): track 23.2 -> 5.61 mm
- net Net-(J1-Pin_4): track 14.3 -> 0.00 mm
- net Net-(J1-Pin_3): track 14.2 -> 0.00 mm
- net Net-(J18-Pin_2): track 20.3 -> 7.64 mm
- net VCC: track 11.9 -> 0.00 mm
- net Net-(U1-GPIO32): track 21.7 -> 10.5 mm
- net +3.3V: track 7.21 -> 16.9 mm
- net Net-(DZ1-A): track 12.8 -> 22.2 mm
- net Net-(U1-GPIO27): track 0.00 -> 7.18 mm
- net Net-(J4-Pin_2): track 35.4 -> 29.2 mm
- net Net-(A1-DIR): track 9.72 -> 4.34 mm
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- removed copper zone on F.Cu, net LINE
- removed copper zone on F.Cu, net VDC

Commit message: -
Parts:
- Q3: value Power Pmos -> IRF9540N
Changed lines of the file:
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@@
 			)
 		)
-		(property "Value" "Power Pmos"
+		(property "Value" "IRF9540N"
 			(at 2.54 2.5 0)
 			(layer "F.Fab")
@@
 		(layer "Edge.Cuts")
 	)
+	(gr_line
+		(start 38.1 86.36)
+		(end 140.97 86.36)
+		(stroke
+			(width 0.1)
+			(type default)
+		)
+		(layer "B.Fab")
+	)
 	(via
